Commit message: Fix gripper mimic sign and add world→base_link leveling joint
Mimic fix (joint7):
- multiplier: -1 → +1
- limits: 0..1.57 → -1.57..0 (must match joint6 range)
Reason: joint6 and joint7 frames differ by π yaw, making their local
Z axes antiparallel in gripper_actuator frame.  Equal joint values
produce opposite physical rotations (symmetric pinch).  The previous
multiplier=-1 inverted this, causing both fingers to sweep the same
world direction.

World joint:
- Added <link name="world"/> + fixed world_joint (world → base_link)
- rpy="0 -0.094954 0" applies a -5.4° corrective pitch derived from
  joint0's SW-exported pitch component (the residual tilt source)
- RViz Fixed Frame changed from base_link to world

File: src/robotic_arm_description/urdf/robotic_arm.urdf.xacro (robot description, xacro)
@@ -12,21 +12,41 @@
     ║                                                               ║
     ║  CHANGES MADE:                                                ║
-    ║  1. joint0 xyz zeroed → arm base sits at world origin.        ║
-    ║  2. joint0 rpy kept unchanged: it encodes the actual physical  ║
+    ║  1. world_joint added (world → base_link, fixed) with a small ║
+    ║     corrective pitch to level the arm on the ground plane.    ║
+    ║     Adjust world_joint rpy pitch if the tilt looks wrong.     ║
+    ║  2. joint0 xyz zeroed → arm base sits at world origin.        ║
+    ║  3. joint0 rpy kept unchanged: it encodes the actual physical ║
     ║     mounting orientation of lower_arm on the base plate.      ║
-    ║     If the arm appears tilted in RViz, verify with hardware   ║
-    ║     and zero rpy if needed.                                   ║
-    ║  3. base_link visual/collision origin shifted by              ║
+    ║  4. base_link visual/collision origin shifted by              ║
     ║     −(joint0_xyz) = (−0.70796, 1.3272, −0.9075) so the base  ║
     ║     plate mesh re-aligns with the arm at world origin.        ║
     ║     (base_link.STL vertices are in SW world coordinates.)     ║
-    ║  4. base_link inertial COM is still in SW world coords —      ║
+    ║  5. base_link inertial COM is still in SW world coords —      ║
     ║     correct it before enabling simulation/dynamics.           ║
-    ║  5. joint6 limits corrected: −1.57..0 (finger closes pos→0). ║
-    ║  6. joint7 limits corrected: 0..1.57, mimic joint6 ×(−1).   ║
-    ║  7. All mesh URIs updated: Robotic_Arm → robotic_arm_description║
-    ║  8. joint1–7 origins: UNTOUCHED (relative transforms exact). ║
+    ║  6. joint6 limits corrected: −1.57..0 (finger closes pos→0). ║
+    ║  7. joint7 limits corrected: −1.57..0, mimic joint6 ×(+1).  ║
+    ║     Multiplier is +1 because joint6/joint7 frames are rotated ║
+    ║     180° in yaw, making their local Z axes antiparallel in    ║
+    ║     the parent frame. Equal joint values → opposite world     ║
+    ║     rotations → symmetric pinch. multiplier=−1 (wrong) caused ║
+    ║     both fingers to rotate in the same world direction.       ║
+    ║  8. All mesh URIs updated: Robotic_Arm → robotic_arm_description║
+    ║  9. joint1–7 origins: UNTOUCHED (relative transforms exact). ║
     ╚═══════════════════════════════════════════════════════════════╝
   -->
+  <!-- ═══════ world ══════════════════════════════════════════════ -->
+  <!-- Massless anchor so RViz/Nav2 have a stable "world" fixed frame. -->
+  <link name="world"/>
+  <!--
+    world_joint — world → base_link  (fixed)
+    The small corrective pitch (−0.095 rad ≈ −5.4°) counteracts the
+    residual tilt from joint0's SW-exported pitch component.
+    Tune this rpy if the arm still looks tilted in RViz.
+  -->
+  <joint name="world_joint" type="fixed">
+    <origin xyz="0 0 0" rpy="0 -0.094954 0"/>
+    <parent link="world"/>
+    <child  link="base_link"/>
+  </joint>
   <!-- ═══════ base_link ═══════════════════════════════════════════ -->
   <link name="base_link">
@@ -324,8 +344,11 @@
     joint7 — gripper_actuator → gripper_2  (right finger)
     CHANGED limits: lower was -0.2, upper was 1.57.
-      Corrected to lower="0" upper="1.57":
-      mirrors joint6; right finger opens toward positive.
-    ADDED mimic: joint7 = −1 × joint6 + 0
-      Both fingers move symmetrically; only joint6 needs a command.
+      Corrected to lower="-1.57" upper="0" (matches joint6).
+    ADDED mimic: joint7 = +1 × joint6 + 0
+      multiplier=+1 because joint6 frame (rpy="...0") and joint7 frame
+      (rpy="...3.1416") are 180° apart in yaw, making their local Z
+      axes antiparallel in the parent frame.  Equal values → opposite
+      physical rotations → symmetric pinch/open.  multiplier=−1 was
+      wrong: it caused both fingers to sweep the same world direction.
     Origin UNCHANGED.
   -->
@@ -335,6 +358,6 @@
     <child  link="gripper_2"/>
     <axis xyz="0 0 1"/>
-    <limit lower="0" upper="1.57" effort="2" velocity="1"/>
-    <mimic joint="joint6" multiplier="-1" offset="0"/>
+    <limit lower="-1.57" upper="0" effort="2" velocity="1"/>
+    <mimic joint="joint6" multiplier="1" offset="0"/>
   </joint>
 </robot>

Commit message: Fix gripper joint limits: lower=-0.093 upper=1.57, positive=open

File: src/robotic_arm_description/urdf/robotic_arm.urdf.xacro (robot description, xacro)
@@ -304,8 +304,7 @@
   <!--
     joint6 — gripper_actuator → gripper_1  (left finger)
-    CHANGED limits: lower was -0.2, upper was 1.57.
-      Corrected to lower="-1.57" upper="0":
-      finger opens toward negative (finger sweeps away from center
-      as joint6 goes negative; fully closed = 0, fully open = -1.57).
+    Positive rotation = finger opens outward.
+    lower="-0.093": almost-closed resting position (slight pre-contact).
+    upper="1.57":   fully open (~90°).
     Origin UNCHANGED.
   -->
@@ -315,5 +314,5 @@
     <child  link="gripper_1"/>
     <axis xyz="0 0 1"/>
-    <limit lower="-1.57" upper="0" effort="2" velocity="1"/>
+    <limit lower="-0.093" upper="1.57" effort="2" velocity="1"/>
   </joint>
   <!-- ═══════ gripper_2 (right finger) ══════════════════════════════ -->
@@ -343,12 +342,9 @@
   <!--
     joint7 — gripper_actuator → gripper_2  (right finger)
-    CHANGED limits: lower was -0.2, upper was 1.57.
-      Corrected to lower="-1.57" upper="0" (matches joint6).
-    ADDED mimic: joint7 = +1 × joint6 + 0
-      multiplier=+1 because joint6 frame (rpy="...0") and joint7 frame
-      (rpy="...3.1416") are 180° apart in yaw, making their local Z
-      axes antiparallel in the parent frame.  Equal values → opposite
-      physical rotations → symmetric pinch/open.  multiplier=−1 was
-      wrong: it caused both fingers to sweep the same world direction.
+    Mirrors joint6 via mimic multiplier=+1.
+    Limits match joint6 exactly: lower="-0.093" upper="1.57".
+    Because joint7's frame is rotated 180° in yaw relative to joint6,
+    equal joint values produce opposite physical rotations → symmetric
+    pinch.  joint6=1.57 AND joint7=1.57 → both fingers open outward.
     Origin UNCHANGED.
   -->
@@ -358,5 +354,5 @@
     <child  link="gripper_2"/>
     <axis xyz="0 0 1"/>
-    <limit lower="-1.57" upper="0" effort="2" velocity="1"/>
+    <limit lower="-0.093" upper="1.57" effort="2" velocity="1"/>
     <mimic joint="joint6" multiplier="1" offset="0"/>
   </joint>

Commit message: Place base plate exactly on world ground plane (z=0)
world_joint xyz: 0 0 0 → 0 0 0.039247
  Derived from base_link.STL Z_min = 0.868253 m (SW coords) minus
  the visual offset Z = -0.9075 m → bottom in base_link = -0.039247 m
  → lift = +0.039247 m → world Z_min = 0.000000 m (verified end-to-end)
  Plate is 5.1 cm thick; top sits at world z = 0.051 m.

world_joint rpy: 0 -0.094954 0 → 0 0 0
  The base plate bottom face is already horizontal in base_link coords
  (square XY extents, Z span = thickness only). The previous pitch
  correction was tilting the plate in world frame, which would cause
  incorrect contact with the Gazebo ground plane.

File: src/robotic_arm_description/urdf/robotic_arm.urdf.xacro (robot description, xacro)
@@ -12,7 +12,7 @@
     ║                                                               ║
     ║  CHANGES MADE:                                                ║
-    ║  1. world_joint added (world → base_link, fixed) with a small ║
-    ║     corrective pitch to level the arm on the ground plane.    ║
-    ║     Adjust world_joint rpy pitch if the tilt looks wrong.     ║
+    ║  1. world_joint added (world → base_link, fixed):             ║
+    ║     z=+0.039247 m lifts base plate bottom to world z=0.       ║
+    ║     rpy=0 0 0 — plate is flat in base_link, no rotation.      ║
     ║  2. joint0 xyz zeroed → arm base sits at world origin.        ║
     ║  3. joint0 rpy kept unchanged: it encodes the actual physical ║
@@ -40,10 +40,17 @@
   <!--
     world_joint — world → base_link  (fixed)
-    The small corrective pitch (−0.095 rad ≈ −5.4°) counteracts the
-    residual tilt from joint0's SW-exported pitch component.
-    Tune this rpy if the arm still looks tilted in RViz.
+    xyz z = +0.039247 m: lifts the robot so the base plate bottom face
+      sits exactly on the world XY ground plane (z = 0).
+      Derived from: base_link.STL Z_min = 0.868253 m (SW coords),
+      visual offset Z = −0.9075 m  →  bottom in base_link = −0.039247 m
+      →  z_lift = 0.039247 m so that −0.039247 + 0.039247 = 0.
+    rpy = 0 0 0: the base plate's bottom face is already horizontal in
+      base_link coords (Z span = 5.1 cm, XY span ≈ 14 cm square), so
+      no rotation is needed to level it on the ground plane.
+      (The previous pitch correction was tilting the plate in world
+      frame, which is wrong for a flat ground spawn.)
   -->
   <joint name="world_joint" type="fixed">
-    <origin xyz="0 0 0" rpy="0 -0.094954 0"/>
+    <origin xyz="0 0 0.039247" rpy="0 0 0"/>
     <parent link="world"/>
     <child  link="base_link"/>

Commit message: Level base plate using PCA plane fit on bottom-face triangles
The base plate was genuinely tilted 8.1° in the SW export — the bottom
face plane normal was [0.0573, 0.1288, 0.9900] in base_link coords,
not [0, 0, 1].  Fitted a least-squares plane to the 17 bottom-face
triangles of base_link.STL, then computed the rotation that maps that
normal onto world Z.

world_joint rpy: 0 0 0 → 0.129355 -0.057284 -0.003711
  (roll 7.4°, pitch −3.3°, yaw −0.2°)

world_joint xyz z: 0.039247 → 0.029710
  Re-derived Z lift after applying the rpy correction so the lowest
  mesh vertex sits exactly at world Z = 0.

Verified: bottom-face world Z = 0.000000 m, flatness deviation = 0.000 mm.

File: src/robotic_arm_description/urdf/robotic_arm.urdf.xacro (robot description, xacro)
@@ -13,6 +13,7 @@
     ║  CHANGES MADE:                                                ║
     ║  1. world_joint added (world → base_link, fixed):             ║
-    ║     z=+0.039247 m lifts base plate bottom to world z=0.       ║
-    ║     rpy=0 0 0 — plate is flat in base_link, no rotation.      ║
+    ║     rpy=0.1294 -0.0573 -0.0037 — derived from PCA plane fit   ║
+    ║     on bottom-face triangles (8.1° tilt in SW export).        ║
+    ║     z=+0.029710 m lifts base plate bottom to world z=0.       ║
     ║  2. joint0 xyz zeroed → arm base sits at world origin.        ║
     ║  3. joint0 rpy kept unchanged: it encodes the actual physical ║
@@ -40,17 +41,18 @@
   <!--
     world_joint — world → base_link  (fixed)
-    xyz z = +0.039247 m: lifts the robot so the base plate bottom face
-      sits exactly on the world XY ground plane (z = 0).
-      Derived from: base_link.STL Z_min = 0.868253 m (SW coords),
-      visual offset Z = −0.9075 m  →  bottom in base_link = −0.039247 m
-      →  z_lift = 0.039247 m so that −0.039247 + 0.039247 = 0.
-    rpy = 0 0 0: the base plate's bottom face is already horizontal in
-      base_link coords (Z span = 5.1 cm, XY span ≈ 14 cm square), so
-      no rotation is needed to level it on the ground plane.
-      (The previous pitch correction was tilting the plate in world
-      frame, which is wrong for a flat ground spawn.)
+    Values derived by fitting a plane to the 17 bottom-face triangles of
+    base_link.STL and computing the rotation that maps the plane normal
+    onto world Z.
+    Bottom-face plane normal in base_link = [0.0573, 0.1288, 0.9900]
+      → 8.1° off vertical in base_link coords (plate is genuinely tilted
+        in the SW export, not just a translation issue).
+    rpy = "0.129355 -0.057284 -0.003711"  (roll 7.4°, pitch −3.3°, yaw −0.2°)
+      Rotates base_link so the bottom face is horizontal in world frame.
+    xyz z = 0.029710 m
+      After applying the rpy, the lowest mesh vertex sits at world Z =
+      −0.029710 m; lifting by that amount places the bottom at z = 0.
   -->
   <joint name="world_joint" type="fixed">
-    <origin xyz="0 0 0.039247" rpy="0 0 0"/>
+    <origin xyz="0 0 0.029710" rpy="0.129355 -0.057284 -0.003711"/>
     <parent link="world"/>
     <child  link="base_link"/>

Commit message: Phase 2: MoveIt 2 config + mock hardware working (ROS 2 Jazzy / MoveIt 2.12.4)
arm_moveit_config
- SRDF: arm chain (joint0-5, base_link→gripper_actuator), gripper group
  (joint6 only — joint7 is passive mimic), named poses home/ready/open/closed,
  all disable_collisions pairs.  No virtual_joint: world_joint already in URDF.
- kinematics.yaml: KDL plugin for arm + gripper groups
- ompl_planning.yaml: RRTConnect default, RRT, PRM configs
- joint_limits.yaml: velocity + acceleration limits for all joints
- moveit_controllers.yaml: MoveItSimpleControllerManager → arm_controller +
  gripper_controller (FollowJointTrajectory)
- ros2_controllers.yaml: JointTrajectoryController × 2 +
  JointStateBroadcaster (ros2_control 4.44)
- moveit.rviz: Fixed Frame = world, MotionPlanning display (not Panel)
- demo.launch.py: RSP + ros2_control_node + controller spawners + move_group
  + RViz2.  Planning pipeline params follow MoveIt 2.12 layout:
  planning_pipelines.pipeline_names=['ompl'] and ompl.planning_plugins=[...]
  at top level (not nested under planning_pipelines — parent_namespace is "").

robotic_arm_description (updates for ros2_control 4.44)
- Added ros2_control block (mock_components/GenericSystem, no deprecated
  fake_sensor_commands / state_following_offset params)
- joint7: mimic joint → state interfaces only, no command interface
  (ros2_control 4.x forbids command interfaces on URDF mimic joints)
- package.xml / CMakeLists.txt: added ros2_control exec_depends

mobile_manipulator_core
- moveit_smoke_test.cpp: (a) move to 'ready', (b) Cartesian target,
  (c) return to 'home' via MoveGroupInterface
- smoke_test.launch.py: runs the test against a live demo session

Verified: planning, execution (SUCCEEDED), and RViz MotionPlanning plugin
all functional with mock hardware.

File: src/robotic_arm_description/urdf/robotic_arm.urdf.xacro (robot description, xacro)
@@ -366,3 +366,68 @@
     <mimic joint="joint6" multiplier="1" offset="0"/>
   </joint>
+  <!-- ═══════ ros2_control hardware interface ══════════════════════
+       mock_components/GenericSystem simulates hardware for the demo.
+       Swap the plugin for a real driver (e.g. serial, EtherCAT) in
+       production.  joint7 is declared as a mimic so controller_manager
+       keeps its state in sync with joint6 automatically.
+  ══════════════════════════════════════════════════════════════════ -->
+  <ros2_control name="robotic_arm_system" type="system">
+    <hardware>
+      <plugin>mock_components/GenericSystem</plugin>
+    </hardware>
+    <joint name="joint0">
+      <command_interface name="position">
+        <param name="min">-3.14</param><param name="max">3.14</param>
+      </command_interface>
+      <state_interface name="position"><param name="initial_value">0.0</param></state_interface>
+      <state_interface name="velocity"><param name="initial_value">0.0</param></state_interface>
+    </joint>
+    <joint name="joint1">
+      <command_interface name="position">
+        <param name="min">-3.14</param><param name="max">3.14</param>
+      </command_interface>
+      <state_interface name="position"><param name="initial_value">0.0</param></state_interface>
+      <state_interface name="velocity"><param name="initial_value">0.0</param></state_interface>
+    </joint>
+    <joint name="joint2">
+      <command_interface name="position">
+        <param name="min">-3.14</param><param name="max">3.14</param>
+      </command_interface>
+      <state_interface name="position"><param name="initial_value">0.0</param></state_interface>
+      <state_interface name="velocity"><param name="initial_value">0.0</param></state_interface>
+    </joint>
+    <joint name="joint3">
+      <command_interface name="position">
+        <param name="min">-3.14</param><param name="max">3.14</param>
+      </command_interface>
+      <state_interface name="position"><param name="initial_value">0.0</param></state_interface>
+      <state_interface name="velocity"><param name="initial_value">0.0</param></state_interface>
+    </joint>
+    <joint name="joint4">
+      <command_interface name="position">
+        <param name="min">-3.14</param><param name="max">3.14</param>
+      </command_interface>
+      <state_interface name="position"><param name="initial_value">0.0</param></state_interface>
+      <state_interface name="velocity"><param name="initial_value">0.0</param></state_interface>
+    </joint>
+    <joint name="joint5">
+      <command_interface name="position">
+        <param name="min">-3.14</param><param name="max">3.14</param>
+      </command_interface>
+      <state_interface name="position"><param name="initial_value">0.0</param></state_interface>
+      <state_interface name="velocity"><param name="initial_value">0.0</param></state_interface>
+    </joint>
+    <joint name="joint6">
+      <command_interface name="position">
+        <param name="min">-0.093</param><param name="max">1.57</param>
+      </command_interface>
+      <state_interface name="position"><param name="initial_value">0.0</param></state_interface>
+      <state_interface name="velocity"><param name="initial_value">0.0</param></state_interface>
+    </joint>
+    <!-- joint7 is a URDF mimic joint: ros2_control 4.x forbids command interfaces on mimic joints. -->
+    <joint name="joint7">
+      <state_interface name="position"><param name="initial_value">0.0</param></state_interface>
+      <state_interface name="velocity"><param name="initial_value">0.0</param></state_interface>
+    </joint>
+  </ros2_control>
 </robot>
