Commit message: Fix Phase 3: wheel inertia (triangle inequality) + DetachableJoint model-level placement
- Wheel ixx=iyy: 4.58e-4 → 1.354e-3 (correct formula m(3r²+h²)/12 for r=0.1,h=0.05)
  Previous values violated ixx+iyy >= izz, causing Gazebo to reject the link
  and preventing gz_ros2_control from starting the controller_manager.
- DetachableJoint plugins moved from world-level to inside each cube model
  (gz::sim::systems::DetachableJoint must be a model plugin, not world plugin)

File: src/mm_bringup/urdf/mobile_base.urdf.xacro (robot description, xacro)
@@ -64,8 +64,11 @@
       <mass value="0.5"/>
       <origin xyz="0 0 0"/>
-      <!-- solid cylinder: Ixx=Iyy=m(3r²+h²)/12  Izz=mr²/2 -->
-      <inertia ixx="4.58e-4" ixy="0" ixz="0"
-               iyy="4.58e-4" iyz="0"
-               izz="2.50e-3"/>
+      <!-- solid cylinder r=0.10 h=0.05 m=0.5:
+           Ixx=Iyy = m(3r²+h²)/12 = 0.5*(0.03+0.0025)/12 = 1.354e-3
+           Izz     = mr²/2        = 0.5*0.01/2            = 2.500e-3
+           Triangle-inequality check: 1.354e-3+1.354e-3 = 2.708e-3 > 2.500e-3 OK -->
+      <inertia ixx="1.354e-3" ixy="0" ixz="0"
+               iyy="1.354e-3" iyz="0"
+               izz="2.500e-3"/>
     </inertial>
   </link>
@@ -87,7 +90,7 @@
       <mass value="0.5"/>
       <origin xyz="0 0 0"/>
-      <inertia ixx="4.58e-4" ixy="0" ixz="0"
-               iyy="4.58e-4" iyz="0"
-               izz="2.50e-3"/>
+      <inertia ixx="1.354e-3" ixy="0" ixz="0"
+               iyy="1.354e-3" iyz="0"
+               izz="2.500e-3"/>
     </inertial>
   </link>

Commit message: Phase 3 verified: SLAM mapping + warehouse walls + sensor fixes
- Fix gz-sim-sensors-system: move to world level in warehouse.sdf (model-scope
  was silently ignored, causing LiDAR to produce no data)
- Remove duplicate Sensors/IMU plugins from mobile_base.urdf.xacro to prevent
  Ogre2 double-scene crash (ItemIdentityException)
- Add perimeter walls to warehouse.sdf so SLAM gets closed boundaries
- Fix SLAM lifecycle: add nav2_lifecycle_manager with autostart to activate
  async_slam_toolbox_node (lifecycle node requires configure+activate)
- Resize mobile base: 0.38x0.30x0.15m, wheel_separation=0.38m in controller
- Switch to DART physics (Bullet Featherstone broke velocity control on wheels)
- Add slam_rviz.rviz config and RViz auto-launch to slam.launch.py
- Set ROS_DOMAIN_ID=42 in .bashrc to isolate from other workspaces
- Save warehouse_map (1074x1262 @ 0.05m/px)

File: src/mm_bringup/urdf/mobile_base.urdf.xacro (robot description, xacro)
@@ -4,8 +4,8 @@
     Mobile differential-drive base for the mobile manipulator.
     Geometry (all from base_footprint which is on the ground):
-      chassis_link  center  z = 0.20 m
-      drive wheels  center  z = 0.10 m  (wheel_radius, bottom at z=0)
-      caster balls  center  z = 0.05 m  (caster_radius, bottom at z=0)
-      chassis top         z = 0.30 m    → arm mounts here
+      chassis_link  center  z = 0.175 m   (box 0.38×0.30×0.15 m)
+      drive wheels  center  z = 0.100 m   (wheel_radius=0.10, bottom at z=0)
+      caster balls  center  z = 0.050 m   (caster_radius=0.05, bottom at z=0)
+      chassis top         z = 0.250 m     → arm mounts here
     The arm is heavy (~8 kg); chassis mass 20 kg keeps CoM low.
   -->
@@ -13,5 +13,5 @@
   <link name="base_footprint"/>
   <joint name="base_footprint_joint" type="fixed">
-    <origin xyz="0 0 0.20" rpy="0 0 0"/>
+    <origin xyz="0 0 0.175" rpy="0 0 0"/>
     <parent link="base_footprint"/>
     <child  link="chassis_link"/>
@@ -20,5 +20,5 @@
     <visual>
       <origin xyz="0 0 0" rpy="0 0 0"/>
-      <geometry><box size="0.50 0.40 0.20"/></geometry>
+      <geometry><box size="0.38 0.30 0.15"/></geometry>
       <material name="dark_grey">
         <color rgba="0.2 0.2 0.2 1.0"/>
@@ -27,18 +27,21 @@
     <collision>
       <origin xyz="0 0 0" rpy="0 0 0"/>
-      <geometry><box size="0.50 0.40 0.20"/></geometry>
-    </collision>
-    <inertial>
-      <!-- 20 kg box: Ixx = m(y²+z²)/12, etc. -->
+      <geometry><box size="0.38 0.30 0.15"/></geometry>
+    </collision>
+    <inertial>
+      <!-- 20 kg box 0.38×0.30×0.15:
+           Ixx = m(y²+z²)/12 = 20*(0.09+0.0225)/12 = 0.188
+           Iyy = m(x²+z²)/12 = 20*(0.1444+0.0225)/12 = 0.278
+           Izz = m(x²+y²)/12 = 20*(0.1444+0.09)/12 = 0.391 -->
       <mass value="20.0"/>
       <origin xyz="0 0 0" rpy="0 0 0"/>
-      <inertia ixx="0.270" ixy="0" ixz="0"
-               iyy="0.438" iyz="0"
-               izz="0.583"/>
+      <inertia ixx="0.188" ixy="0" ixz="0"
+               iyy="0.278" iyz="0"
+               izz="0.391"/>
     </inertial>
   </link>
   <!-- ─── virtual chassis-top link (arm mounting point) ──────────── -->
   <joint name="chassis_top_joint" type="fixed">
-    <origin xyz="0 0 0.10" rpy="0 0 0"/>
+    <origin xyz="0 0 0.075" rpy="0 0 0"/>
     <parent link="chassis_link"/>
     <child  link="chassis_top_link"/>
@@ -46,7 +49,8 @@
   <link name="chassis_top_link"/>
   <!-- ─── drive wheels ────────────────────────────────────────────── -->
-  <!-- wheel_radius=0.10  width=0.05  mass=0.5 kg  axis along Y -->
+  <!-- wheel_radius=0.10  width=0.05  mass=0.5 kg  axis along Y
+       wheel center z = 0.175 - 0.075 = 0.100 m  (bottom at z=0) -->
   <joint name="left_wheel_joint" type="continuous">
-    <origin xyz="0 0.225 -0.10" rpy="-1.5707963 0 0"/>
+    <origin xyz="0 0.190 -0.075" rpy="-1.5707963 0 0"/>
     <parent link="chassis_link"/>
     <child  link="left_wheel_link"/>
@@ -65,7 +69,7 @@
       <origin xyz="0 0 0"/>
       <!-- solid cylinder r=0.10 h=0.05 m=0.5:
-           Ixx=Iyy = m(3r²+h²)/12 = 0.5*(0.03+0.0025)/12 = 1.354e-3
-           Izz     = mr²/2        = 0.5*0.01/2            = 2.500e-3
-           Triangle-inequality check: 1.354e-3+1.354e-3 = 2.708e-3 > 2.500e-3 OK -->
+           Ixx=Iyy = m(3r²+h²)/12 = 1.354e-3
+           Izz     = mr²/2        = 2.500e-3
+           Triangle check: 1.354e-3+1.354e-3 = 2.708e-3 > 2.500e-3 OK -->
       <inertia ixx="1.354e-3" ixy="0" ixz="0"
                iyy="1.354e-3" iyz="0"
@@ -74,5 +78,5 @@
   </link>
   <joint name="right_wheel_joint" type="continuous">
-    <origin xyz="0 -0.225 -0.10" rpy="-1.5707963 0 0"/>
+    <origin xyz="0 -0.190 -0.075" rpy="-1.5707963 0 0"/>
     <parent link="chassis_link"/>
     <child  link="right_wheel_link"/>
@@ -96,7 +100,7 @@
   </link>
   <!-- ─── passive casters (ball, zero friction) ────────────────────── -->
-  <!-- caster_radius=0.05  center at z = 0.05-0.20 = -0.15 from chassis -->
+  <!-- caster_radius=0.05  center z = 0.175-0.125 = 0.050 m  (bottom at z=0) -->
   <joint name="front_caster_joint" type="continuous">
-    <origin xyz="0.20 0 -0.15" rpy="0 0 0"/>
+    <origin xyz="0.15 0 -0.125" rpy="0 0 0"/>
     <parent link="chassis_link"/>
     <child  link="front_caster_link"/>
@@ -114,5 +118,4 @@
       <mass value="0.1"/>
       <origin xyz="0 0 0"/>
-      <!-- solid sphere: I = 2mr²/5 -->
       <inertia ixx="1.0e-4" ixy="0" ixz="0"
                iyy="1.0e-4" iyz="0"
@@ -121,5 +124,5 @@
   </link>
   <joint name="rear_caster_joint" type="continuous">
-    <origin xyz="-0.20 0 -0.15" rpy="0 0 0"/>
+    <origin xyz="-0.15 0 -0.125" rpy="0 0 0"/>
     <parent link="chassis_link"/>
     <child  link="rear_caster_link"/>
@@ -144,5 +147,5 @@
   <!-- ─── LiDAR ─────────────────────────────────────────────────────── -->
   <joint name="lidar_joint" type="fixed">
-    <origin xyz="0.12 0 0.12" rpy="0 0 0"/>
+    <origin xyz="0.10 0 0.09" rpy="0 0 0"/>
     <parent link="chassis_link"/>
     <child  link="lidar_link"/>
@@ -150,5 +153,5 @@
   <link name="lidar_link">
     <visual>
-      <geometry><cylinder radius="0.04" length="0.04"/></geometry>
+      <geometry><cylinder radius="0.035" length="0.04"/></geometry>
       <material name="blue"><color rgba="0.0 0.2 0.8 1.0"/></material>
     </visual>
@@ -174,5 +177,5 @@
   <!-- ─── RGB-D camera on a forward mast ──────────────────────────── -->
   <joint name="camera_mast_joint" type="fixed">
-    <origin xyz="0.20 0 0.12" rpy="0 0 0"/>
+    <origin xyz="0.15 0 0.075" rpy="0 0 0"/>
     <parent link="chassis_link"/>
     <child  link="camera_mast_link"/>
@@ -180,5 +183,5 @@
   <link name="camera_mast_link">
     <visual>
-      <geometry><box size="0.03 0.03 0.25"/></geometry>
+      <geometry><box size="0.025 0.025 0.22"/></geometry>
       <material name="dark_grey"/>
     </visual>
@@ -186,10 +189,10 @@
       <mass value="0.1"/>
       <origin xyz="0 0 0"/>
-      <inertia ixx="5e-4" ixy="0" ixz="0" iyy="5e-4" iyz="0" izz="1e-5"/>
+      <inertia ixx="4e-4" ixy="0" ixz="0" iyy="4e-4" iyz="0" izz="1e-5"/>
     </inertial>
   </link>
   <!-- camera_link: tip of mast, tilted 20° down to see workspace -->
   <joint name="camera_joint" type="fixed">
-    <origin xyz="0.02 0 0.125" rpy="0 0.349 0"/>
+    <origin xyz="0.02 0 0.11" rpy="0 0.349 0"/>
     <parent link="camera_mast_link"/>
     <child  link="camera_link"/>
@@ -197,5 +200,5 @@
   <link name="camera_link">
     <visual>
-      <geometry><box size="0.06 0.12 0.04"/></geometry>
+      <geometry><box size="0.05 0.10 0.035"/></geometry>
       <material name="blue"/>
     </visual>
@@ -234,13 +237,7 @@
     <mu2>1.0</mu2>
   </gazebo>
-  <!-- Sensor system plugins (must be in <gazebo> world-level block) -->
-  <gazebo>
-    <plugin filename="gz-sim-sensors-system"
-            name="gz::sim::systems::Sensors">
-      <render_engine>ogre2</render_engine>
-    </plugin>
-    <plugin filename="gz-sim-imu-system"
-            name="gz::sim::systems::Imu"/>
-  </gazebo>
+  <!-- Sensors system and IMU system are world-level plugins (loaded in warehouse.sdf).
+       They must NOT be here at model scope — Ogre2 would try to create a second
+       render scene and crash with ItemIdentityException. -->
   <!-- 360° 2-D LiDAR → /scan -->
   <gazebo reference="lidar_link">

Commit message: World sizing: resize world from arm URDF measurements + Gazebo Teleop
Table/cubes:
- Table surface lowered 0.81m → 0.38m (arm comfortable pick zone 0.35-0.45m)
- Cube size 50mm → 40mm (65% of ~60mm gripper max opening)
- Cube centres at z=0.40m, y spacing tightened to ±5cm

Camera:
- Mast raised from 0.22m to 0.30m (visual offset), camera at z=0.55m
- Downward tilt 20° → 25° (0.436 rad) — centres frame on table surface

Gazebo Teleop in GUI:
- gz_gui.config: default gz-sim8 plugins + Teleop panel docked
- sim.launch.py: passes --gui-config, adds twist_stamper for teleop
  (gz Twist → /teleop_twist → stamper → /diff_drive_controller/cmd_vel)
- gz_bridge.yaml: bridges /teleop_cmd_vel gz topic → /teleop_twist ROS

Separate cube SDFs (red/green/blue) updated to 40mm to match world.

File: src/mm_bringup/urdf/mobile_base.urdf.xacro (robot description, xacro)
@@ -183,16 +183,18 @@
   <link name="camera_mast_link">
     <visual>
-      <geometry><box size="0.025 0.025 0.22"/></geometry>
+      <origin xyz="0 0 0.15"/>
+      <geometry><box size="0.025 0.025 0.30"/></geometry>
       <material name="dark_grey"/>
     </visual>
     <inertial>
       <mass value="0.1"/>
-      <origin xyz="0 0 0"/>
-      <inertia ixx="4e-4" ixy="0" ixz="0" iyy="4e-4" iyz="0" izz="1e-5"/>
-    </inertial>
-  </link>
-  <!-- camera_link: tip of mast, tilted 20° down to see workspace -->
+      <origin xyz="0 0 0.15"/>
+      <!-- 0.10 kg box 0.025×0.025×0.30: Ixx=Iyy=m(y²+z²)/12≈7.6e-4 -->
+      <inertia ixx="7.6e-4" ixy="0" ixz="0" iyy="7.6e-4" iyz="0" izz="1e-5"/>
+    </inertial>
+  </link>
+  <!-- camera_link: top of mast (z=0.55m), tilted 25° down to see table surface -->
   <joint name="camera_joint" type="fixed">
-    <origin xyz="0.02 0 0.11" rpy="0 0.349 0"/>
+    <origin xyz="0.02 0 0.30" rpy="0 0.436 0"/>
     <parent link="camera_mast_link"/>
     <child  link="camera_link"/>
