Commit message: Phase 6: baseline controller, experiment runner, paper data collection (S3 LLM complete 5/5)
Core infrastructure:
- baseline_controller.cpp: hardcoded 4-step pick-and-deliver (no LLM) with APPROACH_NUDGE_M=0.15
- experiment_runner.cpp + gz_teleport.cpp/.hpp: automated multi-trial runner with world reset
  between trials (cube + arm + base), disturbance injection via /world/warehouse/set_pose
- scenarios.yaml: S1-S5 scenario definitions
- PickAtPose.srv: new service for baseline (bypasses live perception)
- aggregate_results.py: pandas/matplotlib analysis script
- run_full_experiment_matrix.sh: batch runner script

Nav2 / localization:
- Static map approach: map_server + identity map→odom TF (no SLAM drift)
- nav2.launch.py rewritten for static map; nav2_amcl.launch.py added as alternative
- warehouse_map.yaml/pgm updated (corrected origin); warehouse_map_v2 added
- nav2_params.yaml: static_layer+inflation_layer only, MPPI tuning (PreferForwardCritic
  re-enabled, PathAngleCritic forward_preference, xy_goal_tolerance=0.25, vx_min=-0.5)

tool_server_node.cpp fixes:
- drive_back() bug: was measuring unsigned sqrt(dx²+dy²) so forward drift counted as
  "backed up"; now uses signed projection onto backward direction unit vector
- drive_back() speed 0.15→0.25 m/s for better authority against arm reaction forces
- Post-pick sequence: arm home at 25% velocity (slow = small reaction force), then drive_back
- GRASP_STANDOFF 0.03→0.05 m; double-publish grasp with 500ms+1000ms DetachableJoint sleep
- Table collision object in "odom" frame, refreshed at start of every pick_cb
- face_yaw() helper: spins robot to target yaw before Nav2 handoff
- Post-dispatch drive_back(1.0) + face_yaw(0.0) for clean return trip

URDF: wheel joint damping 2.0/0.5 (was 0.3/0.2) to resist arm-induced rotation
planner_node.py: switched back to Anthropic Claude Haiku (Gemini free tier RPM limit unusable)

Paper data: S3 LLM (two-cube sequential) 5/5 complete — 647/545/477/485/601s
Remaining: S1 LLM 4/5, S2 baseline 1/5, S4 baseline 1/5, S5 LLM 0/5

File: src/mm_bringup/urdf/mobile_base.urdf.xacro (robot description, xacro)
@@ -56,4 +56,5 @@
     <child  link="left_wheel_link"/>
     <axis xyz="0 0 1"/>
+    <dynamics damping="2.0" friction="0.5"/>
   </joint>
   <link name="left_wheel_link">
@@ -82,4 +83,5 @@
     <child  link="right_wheel_link"/>
     <axis xyz="0 0 1"/>
+    <dynamics damping="2.0" friction="0.5"/>
   </joint>
   <link name="right_wheel_link">
