Commit message: Phase 4 IK pick/place: arm reaches cube for real grasp
pick() now uses real IK to the detected cube 3-D position:
- Looks up object in /detected_objects; fails if not found
- Opens gripper, moves to pre-grasp 12 cm above cube (MoveIt IK)
- Descends to cube centre; returns {success:false, "out of reach"} if
  either IK step fails — picks can now fail based on actual proximity
- Closes gripper + DetachableJoint attach, lifts 15 cm, retracts home

place() tries IK to location coordinates (PLACE_Z=0.43 m) with
fallback to "ready" pose drop if IK fails.

World geometry adjusted so the arm can reach:
- arm_mount_joint shifted 10 cm forward (xyz="0.10 0 0.029710")
  so arm base is at robot_x+0.10 rather than robot_x
- pick_table replaced with compact front-leg-only shelf at x=2.05
  (no back legs → robot parks at x=1.6 with 4 cm gap to table)
- Cubes moved from x=2.5 to x=2.0; reach from arm at x=1.70:
  sqrt(0.30²+0.05²+0.12²) ≈ 0.33 m << 0.41 m chain length

File: src/mm_bringup/urdf/mobile_manipulator.urdf.xacro (robot description, xacro)
@@ -4,7 +4,8 @@
     Combined mobile manipulator = differential-drive base + 6-DOF arm.
     The arm's world_joint leveling correction (8.1° tilt from PCA plane fit)
-    is preserved in arm_mount_joint with the same xyz/rpy as world_joint:
+    is preserved in arm_mount_joint.  rpy is identical to world_joint.
       rpy = "0.129355 -0.057284 -0.003711"
-      xyz z = 0.029710 m  (base-plate bottom sits flush on chassis top)
+      xyz = "0.10 0 0.029710"  (10 cm forward of chassis centre so the arm
+        can reach objects on the pick table ~30 cm ahead of the parking spot)
     TF chain in simulation:
       map → odom → base_footprint → chassis_link → chassis_top_link
@@ -24,7 +25,9 @@
   <!-- Arm (kinematics only: no world link, no ros2_control block) -->
   <xacro:include filename="$(find robotic_arm_description)/urdf/robotic_arm.urdf.xacro"/>
-  <!-- Mount arm on chassis top, preserving the SW-export leveling correction -->
+  <!-- Mount arm on chassis top, 10 cm forward of centre so the arm reaches
+       objects placed ~30 cm ahead of the robot (cube at x=2.0, robot at x=1.6
+       → arm base at x=1.7, reach needed ≈ 0.33 m < 0.41 m chain length). -->
   <joint name="arm_mount_joint" type="fixed">
-    <origin xyz="0 0 0.029710" rpy="0.129355 -0.057284 -0.003711"/>
+    <origin xyz="0.10 0 0.029710" rpy="0.129355 -0.057284 -0.003711"/>
     <parent link="chassis_top_link"/>
     <child  link="base_link"/>

Commit message: Phase 5: closed-loop LLM task planner (Gemini) — Scenario 1 verified
mm_llm_planner exposes /execute_task: an LLM (Gemini by default, Anthropic
and OpenAI also supported) perceives scene state, chooses and sequences
the Phase 4 tool services via native function-calling, and replans on
tool failures using fresh scene state and error feedback. Logs every
LLM turn and tool call per task for paper data.

Added a 10th tool, drive_distance, for relative base moves that aren't
one of the fixed named locations (odometry-only dead-reckoning, capped
at 2m, reuses the existing /cmd_vel -> diff_drive_controller path).

Scenario 1 ("pick up the red cube and place it in the dispatch zone")
verified end-to-end: 7 LLM turns, 1 replan, ~270s. The replan is a real
demonstration of the closed loop recovering from a failed pick by
navigating, nudging in with drive_distance, and retrying successfully.

Also includes pre-existing uncommitted Phase 4 config updates
(gz_bridge.yaml, mobile_manipulator.urdf.xacro, warehouse.sdf) and the
tool_server_node fixes from this session: removed the duplicate
teleop_stamper that was racing Nav2's twist_stamper on
/diff_drive_controller/cmd_vel, added a retry loop for the pick_table
collision object registration (TF not always ready at startup), and
the finger-midpoint offset correction for pick's grasp targeting.

File: src/mm_bringup/urdf/mobile_manipulator.urdf.xacro (robot description, xacro)
@@ -122,6 +122,22 @@
     </plugin>
   </gazebo>
-  <!-- DetachableJoint plugins for grasping are defined in warehouse.sdf
-       so they have world-level scope and can reference the spawned robot
-       model by name. -->
+  <!-- DetachableJoint plugins for grasping — one per cube colour. Must
+       live here, not in warehouse.sdf: parent_link only resolves within
+       the model the plugin is declared in, and the robot doesn't exist
+       yet when warehouse.sdf loads. -->
+  <xacro:macro name="grasp_joint" params="color">
+    <gazebo>
+      <plugin filename="gz-sim-detachable-joint-system"
+              name="gz::sim::systems::DetachableJoint">
+        <parent_link>gripper_actuator</parent_link>
+        <child_model>${color}_cube</child_model>
+        <child_link>link</child_link>
+        <attach_topic>/grasp/${color}_cube</attach_topic>
+        <detach_topic>/release/${color}_cube</detach_topic>
+      </plugin>
+    </gazebo>
+  </xacro:macro>
+  <xacro:grasp_joint color="red"/>
+  <xacro:grasp_joint color="green"/>
+  <xacro:grasp_joint color="blue"/>
 </robot>
